File: hardware-ESPC3Supermini/ESP32C3_Supermini_LG_climate_contoller.kicad_sch (KiCad schematic)
At the start: 16 parts, among them J1 Conn_01x03_Pin, U1 ESP32-C3_SUPERMINI, U2 TPS560200, U4 TJA1027T

Commit message: # ESP32C3 HW - move to kicad 9 - add some LCSC part numbers
Parts:
- C5: LCSC (none) -> C1525
- J1: LCSC (none) -> C5306495; MPN (none) -> S3B-XH-SM4-TB(LF)(SN)
- L1: JCSC C5289310 -> (none); LCSC (none) -> C5289310
- R1: JCSC C25912 -> (none); LCSC (none) -> C25912
- R2: JCSC C25765 -> (none); LCSC (none) -> C25765
- R3: JCSC C25744 -> (none); LCSC (none) -> C25744
- R4: JCSC C11702 -> (none); LCSC (none) -> C11702
- U2: JCSC C83671 -> (none); LCSC (none) -> C83671
- U4: LCSC (none) -> C194371
Changed lines of the file:
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@@
 (kicad_sch
-	(version 20231120)
+	(version 20250114)
 	(generator "eeschema")
-	(generator_version "8.0")
+	(generator_version "9.0")
 	(paper "A4")
 	(junction
@@
 			)
 		)
-		(property "JCSC" "C25765"
+		(property "LCSC" "C25765"
 			(at 123.19 71.12 0)
 			(effects
@@
 			)
 		)
+		(property "MPN" "S3B-XH-SM4-TB(LF)(SN)"
+			(at 34.29 57.15 0)
+			(effects
+				(font
+					(size 1.27 1.27)
+				)
+				(hide yes)
+			)
+		)
+		(property "LCSC" "C5306495"
+			(at 34.29 57.15 0)
+			(effects
+				(font
+					(size 1.27 1.27)
+				)
+				(hide yes)
+			)
+		)
 		(pin "2"
 		)
@@
 			)
 		)
+		(property "LCSC" "C194371"
+			(at 210.82 48.26 0)
+			(effects
+				(font
+					(size 1.27 1.27)
+				)
+				(hide yes)
+			)
+		)
 		(pin "8"
 		)
@@
 			)
 		)
-		(property "JCSC" "C25912"
+		(property "LCSC" "C25912"
 			(at 123.19 60.96 0)
 			(effects
@@
 			)
 		)
+		(property "LCSC" "C1525"
+			(at 191.77 60.96 0)
+			(effects
+				(font
+					(size 1.27 1.27)
+				)
+				(hide yes)
+			)
+		)
 		(pin "1"
 		)
@@
 			)
 		)
-		(property "JCSC" "C5289310"
+		(property "LCSC" "C5289310"
 			(at 104.14 54.61 90)
 			(effects
@@
 			)
 		)
-		(property "JCSC" "C25744"
+		(property "LCSC" "C25744"
 			(at 185.42 36.83 0)
 			(effects
@@
 			)
 		)
-		(property "JCSC" "C83671"
+		(property "LCSC" "C83671"
 			(at 86.36 57.15 0)
 			(effects
@@
 			)
 		)
-		(property "JCSC" "C11702"
+		(property "LCSC" "C11702"
 			(at 232.41 39.37 0)
 			(effects
@@
 		)
 	)
+	(embedded_fonts no)
 )
